File: Multiboard/_autosave-Multiboard.kicad_pcb (KiCad board)
At the start: 2 copper layers, 150 x 120 mm, 206 parts, among them J1 Conn_01x20_Socket, J2 Conn_01x20_Socket, J3 Debug, J4 USB_C_Receptacle_USB2.0_16P, J5 Conn_01x06_Socket, J6 Conn_02x20_Odd_Even, J7 Conn_02x20_Odd_Even, J8 USB_C_Receptacle_USB2.0_16P, Q1 Q_Dual_NMOS_G1S2G2D2S1D1, Q2 Q_Dual_NMOS_G1S2G2D2S1D1, Q3 Q_Dual_NMOS_G1S2G2D2S1D1, Q4 Q_Dual_NMOS_G1S2G2D2S1D1, Q5 Q_Dual_NMOS_G1S2G2D2S1D1, Q6 Q_Dual_NMOS_G1S2G2D2S1D1, Q7 Q_Dual_NMOS_G1S2G2D2S1D1, SW1 BOOT0, SW2 NRST, SW3 SW_SPST, SW4 SW_SPST, SW5 SW_SPST, SW6 SW_SPST, SW7 KEY, SW8 SW_SPST, U1 STM32F411RET6, U2 MAX662AESA_T, U3 MCP1792x-3302xCB, U4 FT2232HL-REEL, U5 93LCxxC, U6 LCMXO2-1200ZE-1TG144C, U7 FAN1112, U8 NCP1117, Y1 32.768KHz, Y2 25MHz, Y3 12MHz

Commit message: synchronised sch and pcb. Added jtag connection between fpga and ftdi
Parts:
- removed C57, C58, C59, C60, C66: 0.1uF, Capacitor_SMD:C_0603_1608Metric_Pad1.08x0.95mm_HandSolder
- removed C61, C65: 1uF, Capacitor_SMD:C_0603_1608Metric_Pad1.08x0.95mm_HandSolder
- removed C62, C64: 10uF, Capacitor_SMD:C_0603_1608Metric_Pad1.08x0.95mm_HandSolder
- removed C63, C67: 0.01uF, Capacitor_SMD:C_0603_1608Metric_Pad1.08x0.95mm_HandSolder
- C48, C50: value 0.1uF -> 10uF
- C49, C51: value 0.1uF -> 22uF
- C52: value 10uF -> 0.1uF
- C53: value 22uF -> 0.1uF
- C54: value 10uF -> 1uF
- C55: value 22uF -> 10uF
- C56: value 0.1uF -> 0.01uF
- J5: footprint Connector_JST:JST_EH_S6B-EH_1x06_P2.50mm_Horizontal -> Connector_Hirose:Hirose_DF13-06P-1.25DSA_1x06_P1.25mm_Vertical
- R36, R37, R38: value 10k -> 5.1K
- R39: value 10k -> 2.2K
- R40, R41, R42, R64: value 5.1K -> 0
- R43, R62: value 2.2K -> 0
- R44, R54, R57: value 0 -> 2.2K
- R45: value 0 -> 12K 1%
- R46, R47: value 0 -> 10K
- R48: value 2.2K -> 10K
- R49: value 12K 1% -> 0
- R50, R51, R52: value 10K -> 0
- R59, R60: value 0 -> 5.1K
- R61: value 2.2K -> 100
- R63: value 5.1K -> 1K
- R65: value 100 -> 1K
- R66, R68: value 0 -> 1K
- moved R56 375.3 mm to (69.7, 130.5)
- moved R60 369.0 mm to (75.4, 101.9), turned to -90 degrees
- moved R53 368.2 mm to (71.9, 135.7)
- moved R59 367.7 mm to (76.8, 94.6), turned to -90 degrees
- moved R46 357.3 mm to (83.6, 76.2), turned to 90 degrees
- moved R54 355.2 mm to (89.4, 82.0), turned to 90 degrees
- moved R47 354.6 mm to (86.0, 82.9)
- moved R45 352.7 mm to (87.4, 86.7), turned to -90 degrees
- moved R42 351.2 mm to (84.3, 112.3)
- moved R41 347.9 mm to (87.5, 114.2)
- moved R40 345.0 mm to (90.4, 110.0)
- moved R39 332.8 mm to (98.7, 116.8)
- moved R38 332.5 mm to (98.7, 122.8), turned to 180 degrees
- moved R37 332.5 mm to (98.7, 120.6), turned to 180 degrees
- moved R36 332.5 mm to (98.7, 118.5), turned to 180 degrees
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Connections:
- C48 pad 1: 3V3 -> 5V
- C49 pad 1: 3V3 -> VCC_1V2
- C50 pad 1: 3V3 -> 5V
- C51 pad 1: 3V3 -> VCC_3V3
- C52 pad 1: 5V -> VCC_3V3
- C53 pad 1: VCC_1V2 -> 1V2
- C54 pad 1: 5V -> 1V2
- C55 pad 1: VCC_3V3 -> 1V2
- C56 pad 1: VCC_3V3 -> 1V2
- R36 pad 1: PA0-MCU -> 3V3
- R36 pad 2: 3V3 -> PT11D-TMS
- R37 pad 1: PA0-GPIO -> 3V3
- R37 pad 2: Net-(SW6-B) -> PT10D-TDI
- R38 pad 1: PA1-MCU -> 3V3
- R38 pad 2: 3V3 -> PT10C-TDO
- R39 pad 1: PA1-GPIO -> PT11C-TCK
- R39 pad 2: Net-(SW6-B) -> GND
- R40 pad 1: 3V3 -> Net-(U4-ADBUS0)
- R40 pad 2: PT11D-TMS -> PT11C-TCK
- R41 pad 1: 3V3 -> Net-(U4-ADBUS1)
- R42 pad 1: 3V3 -> Net-(U4-ADBUS2)
- R43 pad 1: PT11C-TCK -> Net-(U4-ADBUS3)
- R43 pad 2: GND -> PT11D-TMS
- R44 pad 1: Net-(U4-ADBUS0) -> Net-(U4-~{RESET})
- R44 pad 2: PT11C-TCK -> 3V3
- R45 pad 1: Net-(U4-ADBUS1) -> GND
- R45 pad 2: PT10D-TDI -> Net-(U4-REF)
- R46 pad 1: Net-(U4-ADBUS2) -> Net-(U4-EECS)
- R46 pad 2: PT10C-TDO -> 3V3
- R47 pad 1: Net-(U4-ADBUS3) -> 3V3
- R47 pad 2: PT11D-TMS -> Net-(U4-EEDATA)
- R48 pad 1: Net-(U4-~{RESET}) -> Net-(U5-DO)
- R49 pad 1: GND -> PR10D-Rx
- R49 pad 2: Net-(U4-REF) -> Net-(U4-BDBUS0)
- R50 pad 1: Net-(U4-EECS) -> PR10C-Tx
- R50 pad 2: 3V3 -> Net-(U4-BDBUS1)
- R51 pad 1: 3V3 -> PR10B-RTSn
- R51 pad 2: Net-(U4-EEDATA) -> Net-(U4-BDBUS2)
- R52 pad 1: Net-(U5-DO) -> PR10A-CTSn
- R52 pad 2: 3V3 -> Net-(U4-BDBUS3)
- R53 pad 1: PR10D-Rx -> PR9B-DTRn
- R53 pad 2: Net-(U4-BDBUS0) -> Net-(U4-BDBUS4)
- R54 pad 1: PR10C-Tx -> Net-(U4-EECLK)
- R54 pad 2: Net-(U4-BDBUS1) -> Net-(U5-DO)
- R55 pad 1: PR10B-RTSn -> PR9D-DSRn
- R55 pad 2: Net-(U4-BDBUS2) -> Net-(U4-BDBUS5)
- R56 pad 1: PR10A-CTSn -> PR9C-DCDn
- R56 pad 2: Net-(U4-BDBUS3) -> Net-(U4-BDBUS6)
- R57 pad 1: PR9B-DTRn -> 3V3
- R57 pad 2: Net-(U4-BDBUS4) -> /FPGA/PT12C
- R58 pad 1: Net-(U4-EECLK) -> 3V3
- R58 pad 2: Net-(U5-DO) -> /FPGA/PT12D
- R59 pad 1: PR9D-DSRn -> GND
- R59 pad 2: Net-(U4-BDBUS5) -> Net-(J8-CC1)
- R60 pad 1: PR9C-DCDn -> Net-(J8-CC2)
- R60 pad 2: Net-(U4-BDBUS6) -> GND
- R61 pad 1: 3V3 -> Net-(U7-OUTPUT)
- R61 pad 2: /FPGA/PT12C -> GND
- R62 pad 1: 3V3 -> Net-(U7-OUTPUT)
- R62 pad 2: /FPGA/PT12D -> VCC_1V2
- R63 pad 1: GND -> Net-(D7-A)
- R63 pad 2: Net-(J8-CC1) -> 5V
- R64 pad 1: Net-(J8-CC2) -> Net-(U8-OUTPUT)
- R64 pad 2: GND -> VCC_3V3
- R65 pad 1: Net-(U7-OUTPUT) -> Net-(D8-K)
- R65 pad 2: GND -> 3V3
- R66 pad 1: Net-(U7-OUTPUT) -> Net-(D9-K)
- R66 pad 2: VCC_1V2 -> 3V3
- R67 pad 1: Net-(D7-A) -> Net-(D10-K)
- R67 pad 2: 5V -> 3V3
- R68 pad 1: Net-(U8-OUTPUT) -> Net-(D11-K)
- R68 pad 2: VCC_3V3 -> 3V3
- R69 pad 1: Net-(D8-K) -> Net-(D12-K)
- R70 pad 1: Net-(D9-K) -> Net-(D13-K)
- R71 pad 1: Net-(D10-K) -> Net-(D14-K)
- R72 pad 1: Net-(D11-K) -> Net-(D15-K)
Routing:
- net PT10C-TDO: track 0.00 -> 69.4 mm, vias 0 -> 2
- net PT10D-TDI: track 0.00 -> 64.5 mm, vias 0 -> 2
- net PT11D-TMS: track 0.00 -> 63.5 mm
- net PT11C-TCK: track 0.00 -> 59.2 mm
- net GND: track 146.4 -> 185.5 mm, vias 61 -> 66
- net 3V3: track 133.1 -> 169.2 mm, vias 45 -> 48
- net 5V: track 84.5 -> 98.6 mm, vias 4 -> 8
- net Net-(U4-ADBUS0): track 0.00 -> 10.6 mm, vias 0 -> 2
- net Net-(U4-ADBUS1): track 0.00 -> 10.4 mm
- net Net-(U4-ADBUS2): track 0.00 -> 9.56 mm, vias 0 -> 2
- net 1V2: track 0.00 -> 9.12 mm
- net Net-(U4-ADBUS3): track 0.00 -> 8.07 mm, vias 0 -> 2
- net Net-(U4-EECS): track 15.3 -> 18.8 mm
- net Net-(U4-~{RESET}): track 7.41 -> 8.05 mm
