File: Multiboard/FT2232HL.kicad_sch (KiCad schematic)
At the start: 41 parts, among them J5 Conn_01x06_Socket, U4 FT2232HL-REEL, U5 93LCxxC, Y3 12MHz

Commit message: Fixed glitched nets issue
Parts:
- J5, Y3: now left out of the parts list
- U5: LCSC Part Number (none) -> C1350395
Changed lines of the file:
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@@
 		(unit 1)
 		(exclude_from_sim no)
-		(in_bom yes)
+		(in_bom no)
 		(on_board yes)
 		(dnp no)
@@
 		(unit 1)
 		(exclude_from_sim no)
-		(in_bom yes)
-		(on_board no)
+		(in_bom no)
+		(on_board yes)
 		(dnp no)
 		(fields_autoplaced yes)
@@
 			)
 		)
-		(property "LCSC Part Number" ""
+		(property "LCSC Part Number" "C1350395"
 			(at 40.64 86.36 90)
 			(effects
